File: OAS_PCB/OAS_PCB.sch (KiCad schematic (older format))
At the start: 74 parts, among them U1 TL072

Commit message: fix previous commit uploaded wrong
Parts:
- removed Ct? (x2): 100p, symbol Device:C_Small
- removed Ct? (x2): 1u, symbol Device:C_Small
- removed R? (x4): 100k, symbol Device:R
- removed R? (x2): 1k, symbol Device:R
- removed U? (x3): TL074, symbol Amplifier_Operational:TL074
- added AS? (x3): AS3394, Package_SO:SOIC-24W_7.5x15.4mm_P1.27mm, symbol OAS_PCB-rescue:AS3394-OAS_lib
- added C? (x3): 560p, symbol Device:C_Small
- added C? (x9): 33n, symbol Device:C_Small
- added Cs? (x3): 4.7u, symbol Device:C_Small
- added Cs? (x6): 10u, symbol Device:C_Small
- added Ct? (x3): 2n, symbol Device:C_Small
- added Ct? (x24): 10nF, symbol Device:C_Small
- added D? (x12): DIODE, symbol Simulation_SPICE:DIODE
- added R? (x9): 1k, symbol Device:R
- added R? (x9): 68k, symbol Device:R
- added Rt? (x3): 240k, symbol Device:R
- added U? (x3): CD4051B, symbol Analog_Switch:CD4051B
Connections:
- net 6_ModAmt is gone; now on net cv01: AS?.6 (Mod_Amt_CV)
- net +5V: now also AS?.24 (+Vcc), AS?.24 (+Vcc), AS?.24 (+Vcc)
- net -6.5V: now also AS?.3 (-Vee), AS?.3 (-Vee), AS?.3 (-Vee), Rt?.2, Rt?.2, Rt?.2
- net A0: now also U?.11 (A), U?.11 (A), U?.11 (A)
- net B0: now also U?.10 (B), U?.10 (B), U?.10 (B)
- net C0: now also U?.9 (C), U?.9 (C), U?.9 (C)
- net GND: now also AS?.12 (GND), AS?.12 (GND), AS?.12 (GND), C?.1, C?.1, C?.1, C?.1, C?.1, C?.1, C?.1, C?.1, C?.1, C?.1, C?.1, C?.1, Cs?.1, Cs?.1, Cs?.1, Ct?.2, Ct?.2, Ct?.2, Ct?.2, Ct?.2, Ct?.2, Ct?.2, Ct?.2, Ct?.2, Ct?.2, Ct?.2, Ct?.2, Ct?.2, Ct?.2, Ct?.2, Ct?.2, Ct?.2, Ct?.2, Ct?.2, Ct?.2, Ct?.2, Ct?.2, Ct?.2, Ct?.2, Ct?.2, Ct?.2, Ct?.2, D?.1 (A), D?.1 (A), D?.1 (A), D?.2 (K), D?.2 (K), D?.2 (K), R?.1, R?.1, R?.1, R?.2, R?.2, R?.2, R?.2, R?.2, R?.2
- net PulseOut: now also AS?.5 (D-Trig_Out), AS?.5 (D-Trig_Out), AS?.5 (D-Trig_Out), Cs?.1, Cs?.1, Cs?.1
- net SawtoothOut: now also AS?.9 (Saw_Out), AS?.9 (Saw_Out), AS?.9 (Saw_Out), R?.1, R?.1, R?.1
- net VCA1_In: now also Cs?.1, Cs?.1, Cs?.1, R?.2, R?.2, R?.2
- net VCA2_In: now also Cs?.2, Cs?.2, Cs?.2, R?.1, R?.1, R?.1
- net VCA5_Out: now also AS?.23 (VCA5_Out), AS?.23 (VCA5_Out), AS?.23 (VCA5_Out), R?.1, R?.1, R?.1
- net Wave_OutS1: now also AS?.10 (Wave_Out), AS?.10 (Wave_Out), AS?.10 (Wave_Out), AS?.11 (VCA1), AS?.11 (VCA1), AS?.11 (VCA1), Cs?.2, Cs?.2, Cs?.2, R?.1, R?.1, R?.1, R?.1, R?.1, R?.1
- net cv00: now also AS?.2 (VCO_CV), AS?.2 (VCO_CV), AS?.2 (VCO_CV), Ct?.1, Ct?.1, Ct?.1, U?.13 (X0), U?.13 (X0), U?.13 (X0)
- net cv01: now also AS?.6 (Mod_Amt_CV), AS?.6 (Mod_Amt_CV), AS?.6 (Mod_Amt_CV), Ct?.1, Ct?.1, Ct?.1, U?.14 (X1), U?.14 (X1), U?.14 (X1)
- net cv02: now also AS?.7 (Wave_Sel_CV), AS?.7 (Wave_Sel_CV), AS?.7 (Wave_Sel_CV), Ct?.1, Ct?.1, Ct?.1, U?.15 (X2), U?.15 (X2), U?.15 (X2)
- net cv03: now also AS?.8 (PWM_CV), AS?.8 (PWM_CV), AS?.8 (PWM_CV), Ct?.1, Ct?.1, Ct?.1, U?.12 (X3), U?.12 (X3), U?.12 (X3)
- net cv04: now also AS?.13 (Mix_Bal_CV), AS?.13 (Mix_Bal_CV), AS?.13 (Mix_Bal_CV), Ct?.1, Ct?.1, Ct?.1, U?.1 (X4), U?.1 (X4), U?.1 (X4)
- net cv05: now also AS?.15 (Filt_Res_CV), AS?.15 (Filt_Res_CV), AS?.15 (Filt_Res_CV), Ct?.1, Ct?.1, Ct?.1, U?.5 (X5), U?.5 (X5), U?.5 (X5)
- net cv06: now also AS?.20 (VCF_CV), AS?.20 (VCF_CV), AS?.20 (VCF_CV), Ct?.1, Ct?.1, Ct?.1, U?.2 (X6), U?.2 (X6), U?.2 (X6)
- net cv07: now also AS?.22 (VCA5_CV), AS?.22 (VCA5_CV), AS?.22 (VCA5_CV), Ct?.1, Ct?.1, Ct?.1, U?.4 (X7), U?.4 (X7), U?.4 (X7)
- net at U?.3 (X): now also U?.12 (X3); no longer U?.13 (X0)
- net B1: now reaches U?.10 (B)
- net A1: now reaches U?.11 (A)
- net at U?.14 (X1): now also U?.3 (X)
- net at U?.15 (X2): now also U?.3 (X)
- net at C?.2, R?.2, RV?.1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: now also R?.2, R?.2, R?.2
- net 10_TEENSY_PWM: no longer names the net of U?.10 (8_TX2_IN1)
- net 14_TEENSY_PWM: no longer names the net of U?.21 (14_A0_TX3_SPDIF_OUT)
- net 15_TEENSY_PWM: no longer names the net of U?.22 (15_A1_RX3_SPDIF_IN)
- new net: U?.13 (X0), U?.3 (X)
- new net: AS?.1 (Iref), Rt?.1 (x3)
- new net: AS?.14 (VCA2), R?.2, R?.2 (x3)
- new net: AS?.16 (C1), C?.2 (x3)
- new net: AS?.17 (C2), C?.2 (x3)
- new net: AS?.18 (C3), C?.2 (x3)
- new net: AS?.19 (C4), C?.2 (x3)
- new net: AS?.21 (Cs), Cs?.2, D?.1 (A), D?.2 (K) (x3)
- new net: AS?.4 (Ct), Ct?.1 (x3)
- new net: D?.1 (A), D?.2 (K) (x6)
- no-connect marks 4 -> 7
Other:
- moved on the sheet: DAC?, U?
